Commit message: working on robot tree

File: description/robot_core.xacro (robot description, xacro)
@@ -13,3 +13,51 @@
         <color rgba="0 0 0 1"/>
     </material>
+    <!-- BASE LINK -->
+    <link name = "base_link">
+    </link>
+    <!-- CHASSIS LINK -->
+    <joint name ="chassis_join" type = "fixed">
+        <parent link = "base_link"/>
+        <child link = "chassis"/>
+        <origin xyz = "-0.1 0 0"/>
+    </joint>
+    <link name = "chassis">
+        <visual>
+            <origin xyz = "0.15 0 0.075"/>
+            <geometry>
+                <box size = "0.3 0.3 0.15"/> <!-- The origin of the box will be the centered around the joint.  -->
+            </geometry>
+            <material name = "white"/>
+        </visual>
+    </link>
+    <!-- LEFT WHEEL LINK-->
+    <joint name = "left_wheel_joint" type = "continuous">
+        <parent link = "base_link"/>
+        <child link = "left_wheel"/>
+        <origin xyz = "0 0.175 0" rpy = "-$(pi/2) 0 0"/>
+        <axis xyz = "0 0 1"/>
+    </joint>
+    <link name = "left_wheel">
+        <visual>
+            <geometry>
+                <cylinder radius = "0.05" length = "0.04"/>
+            </geometry>
+            </material name = "blue">
+        </visual>
+    </link>
+    <!-- RIGHT WHEEL LINK-->
+    <joint name = "right_wheel_joint" type = "continuous">
+        <parent link = "base_link"/>
+        <child link = "right_wheel"/>
+        <origin xyz = "0 0.175 0" rpy = "$(pi/2) 0 0"/>
+        <axis xyz = "0 0 -1"/>
+    </joint>
+    <link name = "right_wheel">
+        <visual>
+            <geometry>
+                <cylinder radius = "0.05" length = "0.04"/>
+            </geomtry>
+            </material name = "blue">
+        </visual>
+    </link>
 </robot>
