Commit message: working liDAR and 3D visualization camera

File: description/depth_camera.xacro (robot description, xacro)
@@ -22,5 +22,5 @@
     <gazebo reference="camera_link">
         <material>Gazebo/Red</material>
-        <sensor name="camera" type="camera">
+        <sensor name="camera" type="depth">
             <pose> 0 0 0 0 0 0 </pose>
             <visualize>true</visualize>
@@ -29,5 +29,5 @@
                 <horizontal_fov>1.089</horizontal_fov>
                 <image>
-                    <format>R8G8B8</format>
+                    <format>B8G8R8</format>
                     <width>640</width>
                     <height>480</height>
@@ -40,4 +40,6 @@
             <plugin name="camera_controller" filename="libgazebo_ros_camera.so">
                 <frame_name>camera_link_optical</frame_name>
+                <min_depth>0.1</min_depth>
+                <max_depth>100</max_depth>
             </plugin>
         </sensor>

File: description/lidar.xacro (robot description, xacro)
@@ -26,5 +26,5 @@
         <sensor name="laser" type="ray">
             <pose> 0 0 0 0 0 0 </pose>
-            <visualize>true</visualize>
+            <visualize>false</visualize>
             <update_rate>10</update_rate>
             <ray>
@@ -46,5 +46,5 @@
                 </ros>
                 <output_type>sensor_msgs/LaserScan</output_type>
-                <frame_name>laser_frame</frame_name>
+                <frame_name>laser_frame</frame_name> <!-- scanned distance relative to laser_frame -->
             </plugin>
         </sensor>

File: description/robot.urdf.xacro (robot description, xacro)
@@ -4,4 +4,5 @@
     <xacro:include filename = "gazebo_control.xacro"/>
     <xacro:include filename = "lidar.xacro"/>
-    <xacro:include filename = "camera.xacro"/>
+    <!-- <xacro:include filename = "camera.xacro"/> -->
+    <xacro:include filename = "depth_camera.xacro"/>
 </robot>

File: description/robot_core.xacro (robot description, xacro)
@@ -19,4 +19,12 @@
     <!-- BASE LINK -->
     <link name = "base_link">
+    </link>
+    <!-- BASE_FOOTPRINT LINK -->
+    <joint name = "base_footprint_joint" type = "fixed">
+        <parent link = "base_link"/>
+        <child link = "base_footprint"/>
+        <origin xyz = "0 0 0" rpy = "0 0 0"/>
+    </joint>
+    <link name = "base_footprint">
     </link>
     <!-- CHASSIS LINK -->
@@ -45,7 +53,7 @@
     </link>
     <gazebo reference = "chassis">
-        <material>Gazebo/White</material>
+        <material>Gazebo/White</material> <!-- gazebo is not use a standard URDF <material> tag, but by adding <gazebo>, we are using one of Gazebo's library and telling the simulator to render the link name 'chassis' as white -->
     </gazebo>
-    <!-- LEFT WHEEL LINK-->
+    LEFT WHEEL LINK
     <joint name = "left_wheel_joint" type = "continuous">
         <parent link = "base_link"/>
@@ -77,6 +85,6 @@
         <parent link = "base_link"/>
         <child link = "right_wheel"/>
-        <origin xyz = "0 -0.175 0" rpy = "${pi/2} 0 0"/>
-        <axis xyz = "0 0 -1"/>
+        <origin xyz = "0 -0.175 0" rpy = "${pi/2} 0 0"/> <!-- right hand rule rotation -->
+        <axis xyz = "0 0 -1"/> <!-- set axis of rotation following the right-hand rule. if positive, we want a forward motion of the wheels. -->
     </joint>
     <link name = "right_wheel">
